File: proj05-getting-to-blinky/kicad/proj/proj.kicad_sch (KiCad schematic)
At the start: 7 parts, among them U1 7555

Commit message: getting to blinky in progress
Parts:
- BT1: footprint (none) -> projFootprintLib:S8211-46R
- C1: footprint (none) -> Capacitor_SMD:C_0805_2012Metric_Pad1.18x1.45mm_HandSolder
- D1: footprint (none) -> LED_SMD:LED_0805_2012Metric_Pad1.15x1.40mm_HandSolder
- R1, R2, R3: footprint (none) -> Resistor_SMD:R_0805_2012Metric_Pad1.20x1.40mm_HandSolder
- U1: footprint (none) -> Package_SO:SOIC-8_3.9x4.9mm_P1.27mm; symbol projlib:7555 -> projSymbolLib:7555
Connections:
- net VDD: now reaches BT1.1 (+), R1.1, U1.4 (~RST), U1.8 (VDD)
- net THRES: now reaches C1.1, R2.2, U1.2 (~TRIG), U1.6 (THRES)
- net DISCH: now reaches R1.2, R2.1, U1.7 (DISCH)
Changed lines of the file:
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@@
     (stroke (width 0) (type default) (color 0 0 0 0))
   )
+  (label "DISCH" (at 133.35 77.47 0)
+    (effects (font (size 1.27 1.27)) (justify left bottom))
+  )
+  (label "THRES" (at 134.62 101.6 0)
+    (effects (font (size 1.27 1.27)) (justify left bottom))
+  )
+  (label "VDD" (at 161.29 66.04 0)
+    (effects (font (size 1.27 1.27)) (justify left bottom))
+  )
   (symbol (lib_id "Device:Battery_Cell") (at 104.14 86.36 0) (unit 1)
     (in_bom yes) (on_board yes) (fields_autoplaced)
@@
       (effects (font (size 1.27 1.27)) (justify left))
     )
-    (property "Footprint" "" (id 2) (at 104.14 84.836 90)
+    (property "Footprint" "projFootprintLib:S8211-46R" (id 2) (at 104.14 84.836 90)
       (effects (font (size 1.27 1.27)) hide)
     )
@@
       (effects (font (size 1.27 1.27)) (justify right))
     )
-    (property "Footprint" "" (id 2) (at 190.5 107.95 0)
+    (property "Footprint" "LED_SMD:LED_0805_2012Metric_Pad1.15x1.40mm_HandSolder" (id 2) (at 190.5 107.95 0)
       (effects (font (size 1.27 1.27)) hide)
     )
@@
       (effects (font (size 1.27 1.27)) (justify left))
     )
-    (property "Footprint" "" (id 2) (at 126.6952 114.3 0)
+    (property "Footprint" "Capacitor_SMD:C_0805_2012Metric_Pad1.18x1.45mm_HandSolder" (id 2) (at 126.6952 114.3 0)
       (effects (font (size 1.27 1.27)) hide)
     )
@@
       (effects (font (size 1.27 1.27)) (justify left))
     )
-    (property "Footprint" "" (id 2) (at 188.722 91.44 90)
+    (property "Footprint" "Resistor_SMD:R_0805_2012Metric_Pad1.20x1.40mm_HandSolder" (id 2) (at 188.722 91.44 90)
       (effects (font (size 1.27 1.27)) hide)
     )
@@
     (pin "2")
   )
-  (symbol (lib_id "projlib:7555") (at 161.29 83.82 0) (unit 1)
+  (symbol (lib_id "projSymbolLib:7555") (at 161.29 83.82 0) (unit 1)
     (in_bom yes) (on_board yes)
     (property "Reference" "U1" (id 0) (at 161.29 85.09 0))
     (property "Value" "7555" (id 1) (at 161.29 81.28 0))
-    (property "Footprint" "" (id 2) (at 177.8 109.22 0)
+    (property "Footprint" "Package_SO:SOIC-8_3.9x4.9mm_P1.27mm" (id 2) (at 177.8 109.22 0)
       (effects (font (size 1.27 1.27)) hide)
     )
@@
       (effects (font (size 1.27 1.27)) (justify left))
     )
-    (property "Footprint" "" (id 2) (at 123.952 92.71 90)
+    (property "Footprint" "Resistor_SMD:R_0805_2012Metric_Pad1.20x1.40mm_HandSolder" (id 2) (at 123.952 92.71 90)
       (effects (font (size 1.27 1.27)) hide)
     )
@@
       (effects (font (size 1.27 1.27)) (justify left))
     )
-    (property "Footprint" "" (id 2) (at 123.952 71.12 90)
+    (property "Footprint" "Resistor_SMD:R_0805_2012Metric_Pad1.20x1.40mm_HandSolder" (id 2) (at 123.952 71.12 90)
       (effects (font (size 1.27 1.27)) hide)
     )
@@
     )
     (path "/0e140521-1355-41c7-8e68-dd36649ad71f"
-      (reference "BT1") (unit 1) (value "CR2032") (footprint "")
+      (reference "BT1") (unit 1) (value "CR2032") (footprint "projFootprintLib:S8211-46R")
     )
     (path "/5c7bbb61-9215-4be9-b7e1-c0dedcb8002e"
-      (reference "C1") (unit 1) (value "1u") (footprint "")
+      (reference "C1") (unit 1) (value "1u") (footprint "Capacitor_SMD:C_0805_2012Metric_Pad1.18x1.45mm_HandSolder")
     )
     (path "/2fdd81ed-3592-4f6d-b0ae-fdbad7c5f1f4"
-      (reference "D1") (unit 1) (value "LED") (footprint "")
+      (reference "D1") (unit 1) (value "LED") (footprint "LED_SMD:LED_0805_2012Metric_Pad1.15x1.40mm_HandSolder")
     )
     (path "/b40e69c3-c4f3-4391-bcaa-aa53c5766e26"
-      (reference "R1") (unit 1) (value "1k") (footprint "")
+      (reference "R1") (unit 1) (value "1k") (footprint "Resistor_SMD:R_0805_2012Metric_Pad1.20x1.40mm_HandSolder")
     )
     (path "/a19367d6-645a-483a-b958-46be367025de"
-      (reference "R2") (unit 1) (value "470k") (footprint "")
+      (reference "R2") (unit 1) (value "470k") (footprint "Resistor_SMD:R_0805_2012Metric_Pad1.20x1.40mm_HandSolder")
     )
     (path "/7091d79d-ba23-4c71-b608-b2b72a97f001"
-      (reference "R3") (unit 1) (value "1k") (footprint "")
+      (reference "R3") (unit 1) (value "1k") (footprint "Resistor_SMD:R_0805_2012Metric_Pad1.20x1.40mm_HandSolder")
     )
     (path "/73325b43-57cc-4c1d-9dba-40e4f1f80337"
-      (reference "U1") (unit 1) (value "7555") (footprint "")
-    )
-  )
+      (reference "U1") (unit 1) (value "7555") (footprint "Package_SO:SOIC-8_3.9x4.9mm_P1.27mm")
+    )
+  )
