File: proj05-getting-to-blinky/kicad/proj/proj.kicad_pcb (KiCad board)
At the start: 2 copper layers, 35.6 x 29.2 mm, 7 parts, among them U1 7555

Commit message: pcb done
Routing:
- net /VDD: track 4.22 -> 8.38 mm, vias 0 -> 1
- added copper zone on F.Cu, net /VDD
Other:
- board text added: "AEG"
- board text added: "Getting to Blinky"
