File: proj05-getting-to-blinky/kicad/proj2/proj2.kicad_sch (KiCad schematic)
At the start: 7 parts, among them U1 NTE955MC

Commit message: add footprints to proj05
Parts:
- BT1: footprint (none) -> projFootprintLib:Coin_Cell_Battery_Holder_3V_PN_107_THT
- C1: footprint (none) -> Capacitor_THT:C_Radial_D5.0mm_H11.0mm_P2.00mm
- D1: footprint (none) -> LED_THT:LED_D4.0mm
- R1: footprint (none) -> Resistor_THT:R_Axial_DIN0207_L6.3mm_D2.5mm_P10.16mm_Horizontal
- R2: value 470k -> 100k; footprint (none) -> Resistor_THT:R_Axial_DIN0207_L6.3mm_D2.5mm_P10.16mm_Horizontal
- R3: value 1k -> 470; footprint (none) -> Resistor_THT:R_Axial_DIN0207_L6.3mm_D2.5mm_P10.16mm_Horizontal
- U1: footprint (none) -> Package_DIP:DIP-8_W7.62mm
Changed lines of the file:
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@@
       (effects (font (size 1.27 1.27)) (justify right))
     )
-    (property "Footprint" "" (id 2) (at 158.75 123.19 0)
+    (property "Footprint" "LED_THT:LED_D4.0mm" (id 2) (at 158.75 123.19 0)
       (effects (font (size 1.27 1.27)) hide)
     )
@@
       (effects (font (size 1.27 1.27)) (justify left))
     )
-    (property "Footprint" "" (id 2) (at 96.012 80.01 90)
+    (property "Footprint" "Resistor_THT:R_Axial_DIN0207_L6.3mm_D2.5mm_P10.16mm_Horizontal" (id 2) (at 96.012 80.01 90)
       (effects (font (size 1.27 1.27)) hide)
     )
@@
       (effects (font (size 1.27 1.27)) (justify left))
     )
-    (property "Footprint" "" (id 2) (at 80.01 70.866 90)
+    (property "Footprint" "projFootprintLib:Coin_Cell_Battery_Holder_3V_PN_107_THT" (id 2) (at 80.01 70.866 90)
       (effects (font (size 1.27 1.27)) hide)
     )
@@
       (effects (font (size 1.27 1.27)) (justify left))
     )
-    (property "Value" "470k" (id 1) (at 100.33 99.0599 0)
+    (property "Value" "100k" (id 1) (at 100.33 99.0599 0)
       (effects (font (size 1.27 1.27)) (justify left))
     )
-    (property "Footprint" "" (id 2) (at 96.012 97.79 90)
+    (property "Footprint" "Resistor_THT:R_Axial_DIN0207_L6.3mm_D2.5mm_P10.16mm_Horizontal" (id 2) (at 96.012 97.79 90)
       (effects (font (size 1.27 1.27)) hide)
     )
@@
       (effects (font (size 1.27 1.27)) (justify left))
     )
-    (property "Value" "1k" (id 1) (at 161.29 109.2199 0)
+    (property "Value" "470" (id 1) (at 161.29 109.2199 0)
       (effects (font (size 1.27 1.27)) (justify left))
     )
-    (property "Footprint" "" (id 2) (at 156.972 107.95 90)
+    (property "Footprint" "Resistor_THT:R_Axial_DIN0207_L6.3mm_D2.5mm_P10.16mm_Horizontal" (id 2) (at 156.972 107.95 90)
       (effects (font (size 1.27 1.27)) hide)
     )
@@
       (effects (font (size 1.27 1.27)) (justify left))
     )
-    (property "Footprint" "" (id 2) (at 98.7552 127 0)
+    (property "Footprint" "Capacitor_THT:C_Radial_D5.0mm_H11.0mm_P2.00mm" (id 2) (at 98.7552 127 0)
       (effects (font (size 1.27 1.27)) hide)
     )
@@
     (property "Reference" "U1" (id 0) (at 130.81 99.06 0))
     (property "Value" "NTE955MC" (id 1) (at 132.08 96.52 0))
-    (property "Footprint" "" (id 2) (at 134.366 98.425 0)
+    (property "Footprint" "Package_DIP:DIP-8_W7.62mm" (id 2) (at 134.366 98.425 0)
       (effects (font (size 1.27 1.27)) hide)
     )
@@
     )
     (path "/65a49ee4-9f24-4f18-9633-92c3e5c3f183"
-      (reference "BT1") (unit 1) (value "CR3022") (footprint "")
+      (reference "BT1") (unit 1) (value "CR3022") (footprint "projFootprintLib:Coin_Cell_Battery_Holder_3V_PN_107_THT")
     )
     (path "/c6a82f71-14b0-4875-89fa-23118b5db3bc"
-      (reference "C1") (unit 1) (value "1u") (footprint "")
+      (reference "C1") (unit 1) (value "1u") (footprint "Capacitor_THT:C_Radial_D5.0mm_H11.0mm_P2.00mm")
     )
     (path "/16e150a6-24af-4235-9fa6-76b808ebb5b1"
-      (reference "D1") (unit 1) (value "LED") (footprint "")
+      (reference "D1") (unit 1) (value "LED") (footprint "LED_THT:LED_D4.0mm")
     )
     (path "/581e5d54-1b29-450f-94a8-978d770e026b"
-      (reference "R1") (unit 1) (value "1k") (footprint "")
+      (reference "R1") (unit 1) (value "1k") (footprint "Resistor_THT:R_Axial_DIN0207_L6.3mm_D2.5mm_P10.16mm_Horizontal")
     )
     (path "/82bdafba-adf2-4bd3-9e80-820554f930f2"
-      (reference "R2") (unit 1) (value "470k") (footprint "")
+      (reference "R2") (unit 1) (value "100k") (footprint "Resistor_THT:R_Axial_DIN0207_L6.3mm_D2.5mm_P10.16mm_Horizontal")
     )
     (path "/ba9f3286-c922-4834-94fb-1ec8cc5afcdb"
-      (reference "R3") (unit 1) (value "1k") (footprint "")
+      (reference "R3") (unit 1) (value "470") (footprint "Resistor_THT:R_Axial_DIN0207_L6.3mm_D2.5mm_P10.16mm_Horizontal")
     )
     (path "/eca6244e-5791-4275-b150-fb37c20caf6c"
-      (reference "U1") (unit 1) (value "NTE955MC") (footprint "")
+      (reference "U1") (unit 1) (value "NTE955MC") (footprint "Package_DIP:DIP-8_W7.62mm")
     )
   )

Commit message: pcb layout proj05
Changed lines of the file:
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@@
   (junction (at 97.79 135.2804) (diameter 0) (color 0 0 0 0)
+  )
+  (junction (at 132.842 84.2772) (diameter 0) (color 0 0 0 0)
   )
   (junction (at 97.79 90.3224) (diameter 0) (color 0 0 0 0)
@@
   )
   (junction (at 128.905 135.2804) (diameter 0) (color 0 0 0 0)
-  )
-  (junction (at 132.842 84.328) (diameter 0) (color 0 0 0 0)
   )
   (junction (at 97.79 76.2) (diameter 0) (color 0 0 0 0)
@@
     (stroke (width 0) (type default) (color 0 0 0 0))
   )
-  (wire (pts (xy 132.842 65.0494) (xy 132.842 84.328))
+  (wire (pts (xy 132.842 65.0494) (xy 132.842 84.2772))
     (stroke (width 0) (type default) (color 0 0 0 0))
   )
@@
     (stroke (width 0) (type default) (color 0 0 0 0))
   )
-  (wire (pts (xy 132.842 84.328) (xy 132.842 86.741))
+  (wire (pts (xy 132.842 84.2772) (xy 132.842 86.741))
     (stroke (width 0) (type default) (color 0 0 0 0))
   )
@@
     (stroke (width 0) (type default) (color 0 0 0 0))
   )
-  (wire (pts (xy 128.905 84.2772) (xy 132.842 84.328))
+  (wire (pts (xy 128.905 84.2264) (xy 132.842 84.2772))
     (stroke (width 0) (type default) (color 0 0 0 0))
   )
@@
     (stroke (width 0) (type default) (color 0 0 0 0))
   )
-  (wire (pts (xy 128.905 86.741) (xy 128.905 84.2772))
+  (wire (pts (xy 128.905 86.741) (xy 128.905 84.2264))
     (stroke (width 0) (type default) (color 0 0 0 0))
   )
@@
     (stroke (width 0) (type default) (color 0 0 0 0))
   )
+  (label "VDD" (at 79.9592 68.7324 0)
+    (effects (font (size 1.27 1.27)) (justify left bottom))
+  )
+  (label "GND" (at 129.0574 124.3838 0)
+    (effects (font (size 1.27 1.27)) (justify left bottom))
+  )
+  (label "Disch" (at 107.2388 90.4748 0)
+    (effects (font (size 1.27 1.27)) (justify left bottom))
+  )
+  (label "VDD" (at 132.7912 87.0966 0)
+    (effects (font (size 1.27 1.27)) (justify left bottom))
+  )
+  (label "Thres" (at 107.6706 111.633 0)
+    (effects (font (size 1.27 1.27)) (justify left bottom))
+  )
   (symbol (lib_id "power:PWR_FLAG") (at 112.5474 65.0494 0) (unit 1)

Commit message: add mounting holes proj5
Parts:
- added H1, H2, H3: MountingHole, MountingHole:MountingHole_3mm, symbol Mechanical:MountingHole
Other:
- note added: "Mounting Holes"
Changed lines of the file:
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@@
     (stroke (width 0) (type default) (color 0 0 0 0))
+  )
+  (text "Mounting Holes" (at 177.6222 65.659 0)
+    (effects (font (size 1.27 1.27)) (justify left bottom))
   )
   (label "VDD" (at 79.9592 68.7324 0)
@@
     (pin "2")
   )
+  (symbol (lib_id "Mechanical:MountingHole") (at 179.07 81.661 0) (unit 1)
+    (in_bom yes) (on_board yes) (fields_autoplaced)
+    (property "Reference" "H3" (id 0) (at 181.8132 80.3909 0)
+      (effects (font (size 1.27 1.27)) (justify left))
+    )
+    (property "Value" "MountingHole" (id 1) (at 181.8132 82.9309 0)
+      (effects (font (size 1.27 1.27)) (justify left))
+    )
+    (property "Footprint" "MountingHole:MountingHole_3mm" (id 2) (at 179.07 81.661 0)
+      (effects (font (size 1.27 1.27)) hide)
+    )
+    (property "Datasheet" "~" (id 3) (at 179.07 81.661 0)
+      (effects (font (size 1.27 1.27)) hide)
+    )
+  )
   (symbol (lib_id "Device:R") (at 97.79 80.01 0) (unit 1)
     (in_bom yes) (on_board yes) (fields_autoplaced)
@@
     (pin "2")
   )
+  (symbol (lib_id "Mechanical:MountingHole") (at 178.9938 75.9968 0) (unit 1)
+    (in_bom yes) (on_board yes) (fields_autoplaced)
+    (property "Reference" "H2" (id 0) (at 181.991 74.7267 0)
+      (effects (font (size 1.27 1.27)) (justify left))
+    )
+    (property "Value" "MountingHole" (id 1) (at 181.991 77.2667 0)
+      (effects (font (size 1.27 1.27)) (justify left))
+    )
+    (property "Footprint" "MountingHole:MountingHole_3mm" (id 2) (at 178.9938 75.9968 0)
+      (effects (font (size 1.27 1.27)) hide)
+    )
+    (property "Datasheet" "~" (id 3) (at 178.9938 75.9968 0)
+      (effects (font (size 1.27 1.27)) hide)
+    )
+  )
   (symbol (lib_id "power:PWR_FLAG") (at 109.601 135.2804 0) (unit 1)
     (in_bom yes) (on_board yes) (fields_autoplaced)
@@
     (pin "1")
     (pin "2")
+  )
+  (symbol (lib_id "Mechanical:MountingHole") (at 178.9938 70.0786 0) (unit 1)
+    (in_bom yes) (on_board yes) (fields_autoplaced)
+    (property "Reference" "H1" (id 0) (at 182.2196 68.8085 0)
+      (effects (font (size 1.27 1.27)) (justify left))
+    )
+    (property "Value" "MountingHole" (id 1) (at 182.2196 71.3485 0)
+      (effects (font (size 1.27 1.27)) (justify left))
+    )
+    (property "Footprint" "MountingHole:MountingHole_3mm" (id 2) (at 178.9938 70.0786 0)
+      (effects (font (size 1.27 1.27)) hide)
+    )
+    (property "Datasheet" "~" (id 3) (at 178.9938 70.0786 0)
+      (effects (font (size 1.27 1.27)) hide)
+    )
   )
   (symbol (lib_id "projSymbolLib:NTE955MC") (at 130.81 97.79 0) (unit 1)
@@
       (reference "D1") (unit 1) (value "LED") (footprint "LED_THT:LED_D4.0mm")
     )
+    (path "/cae56f63-c338-4b20-bfbb-0a7849b4241e"
+      (reference "H1") (unit 1) (value "MountingHole") (footprint "MountingHole:MountingHole_3mm")
+    )
+    (path "/8771a73d-f63d-4796-98f2-61c4fd4d63bb"
+      (reference "H2") (unit 1) (value "MountingHole") (footprint "MountingHole:MountingHole_3mm")
+    )
+    (path "/4a26099b-912b-4395-97c7-41968a0f921e"
+      (reference "H3") (unit 1) (value "MountingHole") (footprint "MountingHole:MountingHole_3mm")
+    )
     (path "/581e5d54-1b29-450f-94a8-978d770e026b"
