File: proj07-astrostepper-oled/kicad/proj/proj.kicad_sch (KiCad schematic)
At the start: 3 parts

Commit message: kicad start proj07
Parts:
- M?: value Stepper_Motor_bipolar -> Nema 17 Stepper Motor Bipolar 0.9deg; Notes (none) -> STEPPERONLINE 0.9deg Nema 17 Stepper Motor Bipolar 0.9A 36N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
Changed lines of the file:
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@@
 (kicad_sch (version 20211123) (generator eeschema)
   (paper "A4")
+  (symbol (lib_id "power:GND") (at 116.84 109.22 0) (unit 1)
+    (in_bom yes) (on_board yes) (fields_autoplaced)
+    (property "Reference" "#PWR?" (id 0) (at 116.84 115.57 0)
+      (effects (font (size 1.27 1.27)) hide)
+    )
+    (property "Value" "GND" (id 1) (at 116.84 114.3 0))
+    (property "Footprint" "" (id 2) (at 116.84 109.22 0)
+      (effects (font (size 1.27 1.27)) hide)
+    )
+    (property "Datasheet" "" (id 3) (at 116.84 109.22 0)
+      (effects (font (size 1.27 1.27)) hide)
+    )
+    (pin "1")
+  )
   (symbol (lib_id "Motor:Stepper_Motor_bipolar") (at 210.82 57.15 0) (unit 1)
-    (in_bom yes) (on_board yes) (fields_autoplaced)
+    (in_bom yes) (on_board yes)
     (property "Reference" "M?" (id 0) (at 215.9 55.029 0)
       (effects (font (size 1.27 1.27)) (justify left))
     )
-    (property "Value" "Stepper_Motor_bipolar" (id 1) (at 215.9 57.569 0)
+    (property "Value" "Nema 17 Stepper Motor Bipolar 0.9deg" (id 1) (at 193.04 66.04 0)
       (effects (font (size 1.27 1.27)) (justify left))
     )
@@
       (effects (font (size 1.27 1.27)) hide)
     )
-    (property "Datasheet" "http://www.infineon.com/dgdl/Application-Note-TLE8110EE_driving_UniPolarStepperMotor_V1.1.pdf?fileId=db3a30431be39b97011be5d0aa0a00b0" (id 3) (at 211.074 57.404 0)
+    (property "Datasheet" "https://m.media-amazon.com/images/I/91YX52MvwaL.pdf" (id 3) (at 211.074 57.404 0)
+      (effects (font (size 1.27 1.27)) hide)
+    )
+    (property "Notes" "STEPPERONLINE 0.9deg Nema 17 Stepper Motor Bipolar 0.9A 36Ncm/50oz.in 42x42x39mm 4-wires DIY  17HM15-0904S OSM 20161018" (id 4) (at 210.82 57.15 0)
       (effects (font (size 1.27 1.27)) hide)
     )
@@
     (pin "8")
     (pin "9")
+  )
+  (symbol (lib_id "power:+5V") (at 78.74 121.92 0) (unit 1)
+    (in_bom yes) (on_board yes) (fields_autoplaced)
+    (property "Reference" "#PWR?" (id 0) (at 78.74 125.73 0)
+      (effects (font (size 1.27 1.27)) hide)
+    )
+    (property "Value" "+5V" (id 1) (at 78.74 116.84 0))
+    (property "Footprint" "" (id 2) (at 78.74 121.92 0)
+      (effects (font (size 1.27 1.27)) hide)
+    )
+    (property "Datasheet" "" (id 3) (at 78.74 121.92 0)
+      (effects (font (size 1.27 1.27)) hide)
+    )
+    (pin "1")
+  )
+  (symbol (lib_id "power:+7.5V") (at 158.75 101.6 0) (unit 1)
+    (in_bom yes) (on_board yes) (fields_autoplaced)
+    (property "Reference" "#PWR?" (id 0) (at 158.75 105.41 0)
+      (effects (font (size 1.27 1.27)) hide)
+    )
+    (property "Value" "+7.5V" (id 1) (at 158.75 96.52 0))
+    (property "Footprint" "" (id 2) (at 158.75 101.6 0)
+      (effects (font (size 1.27 1.27)) hide)
+    )
+    (property "Datasheet" "" (id 3) (at 158.75 101.6 0)
+      (effects (font (size 1.27 1.27)) hide)
+    )
+    (pin "1")
   )
   (symbol (lib_id "RF_Module:ESP32-WROOM-32D") (at 58.42 78.74 0) (unit 1)
@@
   )
   (symbol_instances
+    (path "/01036636-e400-4fa1-be0a-7c0d6af3db56"
+      (reference "#PWR?") (unit 1) (value "GND") (footprint "")
+    )
+    (path "/c23999d6-11a5-481a-95da-0e4523912ae2"
+      (reference "#PWR?") (unit 1) (value "+5V") (footprint "")
+    )
+    (path "/c4e665d9-0026-4a12-99ce-1740d93782bd"
+      (reference "#PWR?") (unit 1) (value "+7.5V") (footprint "")
+    )
     (path "/0af28087-7f8d-4214-bc65-72d3c31bf4bb"
-      (reference "M?") (unit 1) (value "Stepper_Motor_bipolar") (footprint "")
+      (reference "M?") (unit 1) (value "Nema 17 Stepper Motor Bipolar 0.9deg") (footprint "")
     )
     (path "/a1bc0026-c979-4bcf-ac28-2fdcb44b0d4b"

Commit message: proj07 stepper is working
Parts:
- removed U?: L298N, Package_TO_SOT_THT:TO-220-15_P2.54x2.54mm_StaggerOdd_Lead4.58mm_Vertical, symbol Driver_Motor:L298N
- added U2: L298N_Moter_Driver, symbol projSymbolLib:L298N_Moter_Driver
- gave numbers to parts that had none: 2
Connections:
- net +5V: now also U1.2 (VDD), U2.11 (5v)
- net +7.5V: now also U2.9 (vms)
- net GND: now also U1.1 (GND), U1.15 (GND), U1.38 (GND), U1.39 (GND), U2.10 (GND)
- net at M1.1: now also U2.4 (out4)
- net at M1.2 (-): now also U2.3 (out3)
- net at M1.3: now also U2.2 (out2)
- net at M1.4: now also U2.1 (out1)
- net at U1.10 (IO25): now also U2.5 (in1)
- net at U1.11 (IO26): now also U2.6 (in2)
- net at U1.8 (IO32): now also U2.7 (in3)
- net at U1.9 (IO33): now also U2.8 (in4)
- no-connect marks 0 -> 29
Other:
- title: (none) -> Astrostepper plus OLED
- moved on the sheet: M1, U1
